File: TDA7267/TDA7267.kicad_pcb (KiCad board)
At the start: 2 copper layers, 43 x 39 mm, 18 parts, among them U1 TDA7267

Commit message: Improvements
Parts:
- moved H3 4.50 mm to (132.0, 108.0)
- moved C4 3.80 mm to (135.5, 100.4), turned to 180 degrees
- moved RV1 0.25 mm to (145.0, 114.8)
Routing:
- net Net-(U1-V+): track 46.0 -> 43.3 mm
- net Net-(IN1-Pin_1): track 20.9 -> 19.5 mm
- net Net-(U1-SRV): track 14.6 -> 15.3 mm

Commit message: Tweaks
Parts:
- C1: footprint Capacitor_THT:C_Disc_D6.0mm_W2.5mm_P5.00mm -> Capacitor_THT:C_Rect_L7.2mm_W3.5mm_P5.00mm_FKS2_FKP2_MKS2_MKP2
- moved C2 5.68 mm to (164.8, 100.6)
- moved C3 2.07 mm to (141.7, 103.6)
- moved R1 2.07 mm to (146.7, 105.1)
- moved C1 1.56 mm to (157.1, 105.3)
- renumbered U1 to TDA7267
Routing:
- net Net-(U1-V+): track 43.3 -> 0.00 mm
- net Net-(IN1-Pin_1): track 19.5 -> 0.00 mm
- net Net-(U1-Out): track 17.3 -> 0.00 mm
- net Net-(OUT1-Pin_1): track 17.0 -> 0.00 mm
- net Net-(U1-SRV): track 15.3 -> 0.00 mm
- net Net-(C1-Pad1): track 11.4 -> 0.00 mm
- net Net-(U1-In): track 11.0 -> 0.00 mm
- net Net-(D1-A): track 5.64 -> 0.00 mm
- net Net-(C1-Pad2): track 5.04 -> 0.00 mm
Other:
- board size 43 x 39 mm -> 43 x 31 mm

Commit message: Tweaks
Routing:
- net Net-(U1-V+): track 0.00 -> 43.3 mm
- net Net-(IN1-Pin_1): track 0.00 -> 19.5 mm
- net Net-(U1-SRV): track 0.00 -> 17.7 mm
- net Net-(U1-Out): track 0.00 -> 17.3 mm
- net Net-(OUT1-Pin_1): track 0.00 -> 17.0 mm
- net Net-(C1-Pad1): track 0.00 -> 12.4 mm
- net Net-(U1-In): track 0.00 -> 10.00 mm
- net Net-(D1-A): track 0.00 -> 5.64 mm
- net Net-(C1-Pad2): track 0.00 -> 5.45 mm
Other:
- board size 43 x 31 mm -> 43 x 39 mm
